Commit message: Update arduino_robot_arm.urdf

File: arduino_robot_arm-main/robot_arm_pkg/urdf/arduino_robot_arm.urdf (robot description, URDF)
Before this commit: robot arduino_robot_arm, 5 links, 4 joints
Links:
- removed link arm1
- removed link arm2
- added link 3, mass 0.001; collision box size=0.04221 0.16277 0.02051; visual mesh filename=package://robot_arm_pkg/meshes/stl/4.stl scale=0.00098 0.00098 0.00098
- added link 4, mass 0.001; collision box size=0.02681 0.16397 0.0384; visual mesh filename=package://robot_arm_pkg/meshes/stl/5.stl scale=0.00098 0.00098 0.00098
- link base: geometry collision cylinder length=0.05469 radius=0.0592; visual mesh filename=package://robot_arm_pkg/meshes/stl/1.stl scale=0.00098 0.00098 0.00098
- link gripper: geometry collision mesh filename=package://robot_arm_pkg/meshes/stl/all.stl scale=0.00391 0.00391 0.00391; visual mesh filename=package://robot_arm_pkg/meshes/stl/7.stl scale=0.00391 0.00391 0.00391
- link waist: geometry collision mesh filename=package://robot_arm_pkg/meshes/stl/3.stl scale=0.00391 0.00391 0.00391; visual mesh filename=package://robot_arm_pkg/meshes/stl/2.stl scale=0.00098 0.00098 0.00098
Joints:
- removed joint base_joint
- added joint all: type revolute, parent base, child waist, origin xyz=-0.00345 -1e-05 0.04449 rpy=0 0 0, axis 0 0 1.0, limit lower=-1.571 upper=1.571 effort=1000.0 velocity=1.0
